File: Hardware/Kicad/TRH9000/TRH9000_VIDEO.kicad_sch (KiCad schematic)
At the start: 35 parts, among them J1 RGB, J2 Console5_SCART, Q1 BC817, U6 LMH1980

Commit message: Started routing the PCB, adding cut-outs to separate the analog from digital signal-domains.
Parts:
- removed C17, C19, C20, C21: 220uF, Capacitor_THT:CP_Radial_D5.0mm_P2.50mm, symbol Device:C_Polarized
- added C17, C19, C20, C21: C_TCJB227, Capacitor_Tantalum_SMD:CP_EIA-3528-15_AVX-H, symbol LRJ-parts:C_TCJB227
- added C2, C24: C_CC0805JPX7R9BB104, Capacitor_SMD:C_0805_2012Metric, symbol LRJ-parts:C_CC0805JPX7R9BB104
- added C25: C_GRM188D71A106KA73D, Capacitor_SMD:C_0603_1608Metric, symbol LRJ-parts:C_GRM188D71A106KA73D
- added C40: 47pF, Capacitor_SMD:C_0603_1608Metric, symbol Device:C
- added R11: R_ERJ-3GEYJ105V, Resistor_SMD:R_0603_1608Metric, symbol LRJ-parts:R_ERJ-3GEYJ105V
Connections:
- net BOUT: now also C21.2
- net GND: now also C2.2, C24.2, C25.1, C40.2, R11.1; no longer J2.14 (DATGND), J2.18 (BLNKGND), J2.21 (SH)
- net GOUT: now also C20.2
- net ROUT: now also C19.2
- net BO_: now reaches R19.1
- net BO_: now also C21.1
- net at Q1.2 (E), R13.1: now also C17.1
- net VSOUT: now reaches R26.2, U6.7 (VSOUT)
- net RO_: now reaches R17.1
- net RO_: now also C19.1
- net at R15.2: now also C17.2
- net HSOUT: now reaches R25.2, U6.6 (HSOUT)
- net GO_: now reaches R18.1
- net GO_: now also C20.1
- net REXT: now reaches R24.2, U6.1 (REXT)
- net +12V renamed +12VA
- net +5V renamed +5VA
- net 2.5V renamed 2.5VA
- net GND1 renamed GNDD
- removed net GNDA: J1.6 (GNDr), J1.7 (GNDg), J1.8 (GNDb), J2.13 (RGND), J2.17 (VGND), J2.4 (AUGND), J2.5 (BGND), J2.9 (GGND)
- net SYNCIN renamed Csync_
- new net: C25.2, J2.14 (DATGND), J2.18 (BLNKGND), J2.4 (AUGND)
- new net: C40.1, J2.17 (VGND)
- new net: J2.21 (SH), R11.2
- new net Col_GND: C24.1, J2.13 (RGND), J2.5 (BGND), J2.9 (GGND)
- new net VGA_GND: C2.1, J1.6 (GNDr), J1.7 (GNDg), J1.8 (GNDb)
Other:
- note added: "1. RGB-input"
- note added: "2. CSync Amplifier"
- note added: "3. Sync Separator"
- note added: "4. Video Output Connectors"
- note removed: "CSync Amplifier"
- note removed: "Sync Separator"
- note removed: "Video Output Connectors"
- moved on the sheet: C13, C32, C33, C34, J1, J2, Q1, R10, R12, R13, R15, R17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
