File: Hardware/Kicad/TRH9000/TRH9000_VIDEO.kicad_sch (KiCad schematic)
At the start: 33 parts, among them J1 RGB, J2 S-Video, Q1 BC817, U6 CXA2075M

Commit message: Merging in most recent upstream changes.
Parts:
- removed C13: 47pF, Capacitor_THT:CP_Radial_D5.0mm_P2.50mm, symbol Device:C_Polarized
- removed C18: 47pF, Capacitor_SMD:C_0805_2012Metric, symbol Device:C
- removed C22, C23, C24: 220uF, Capacitor_THT:CP_Radial_D5.0mm_P2.50mm, symbol Device:C_Polarized
- removed J1: RGB, Connector_Dsub:DSUB-15-HD_Female_Horizontal_P2.29x1.98mm_EdgePinOffset3.03mm_Housed_MountingHolesOffset4.94mm, symbol Connector:DB15_Female_HighDensity
- removed J2: S-Video, Connector_PinHeader_2.54mm:PinHeader_1x04_P2.54mm_Vertical, symbol Connector:Mini-DIN-4
- removed R11: 4K7, Resistor_SMD:R_0805_2012Metric, symbol Device:R
- removed R14, R8: 2K2, Resistor_SMD:R_0805_2012Metric, symbol Device:R
- removed R16: 2K61, Resistor_SMD:R_0805_2012Metric, symbol Device:R
- removed R20: 43R, Resistor_SMD:R_0805_2012Metric, symbol Device:R
- removed R21, R22: 75R, Resistor_SMD:R_0805_2012Metric, symbol Device:R
- removed R23: 240R, Resistor_SMD:R_0805_2012Metric, symbol Device:R
- removed U6: CXA2075M, Package_SO:SOP-24_7.5x15.4mm_P1.27mm, symbol TRH9000:CXA2075M
- added C13: 10µF, Capacitor_SMD:C_0805_2012Metric, symbol LRJ-parts:C_GRM188D71A106KA73D
- added C32, C33: 47pF, Capacitor_SMD:C_0805_2012Metric, symbol Device:C
- added C34: 0.1µF, Capacitor_SMD:C_0805_2012Metric, symbol LRJ-parts:C_CL10B104KB8NNNL
- added J1: RGB, Connector_Dsub:DSUB-15-HD_Female_Horizontal_P2.29x1.98mm_EdgePinOffset3.03mm_Housed_MountingHolesOffset4.94mm, symbol Connector:DB15_Female
- added J2: Console5_SCART, LRJ:SCART-21_Female_Horizontal_P1.905x2.54mm_EdgePinOffset10.7mm, symbol LRJ-parts:Console5_SCART
- added R10, R25, R26: 100, Resistor_SMD:R_0805_2012Metric, symbol Device:R
- added R24: 10k, Capacitor_SMD:C_0805_2012Metric, symbol LRJ-parts:R_RC0603FR-0710KL
- added R27, R28: 100, Resistor_SMD:R_0603_1608Metric, symbol Device:R
- added R29: 1k, Resistor_SMD:R_0603_1608Metric, symbol Device:R
- added R9: 75, Resistor_SMD:R_0805_2012Metric, symbol Device:R
- added U6: LMH1980, Package_SO:VSSOP-10_3x3mm_P0.5mm, symbol LRJ-parts:LMH1980
Connections:
- net +5V: now also R27.1
- net BOUT: now also J1.3, J2.7 (BLUE)
- net GND: now also C13.1, C32.2, C33.2, J2.14 (DATGND), J2.18 (BLNKGND), J2.21 (SH), R24.1, R28.2, R9.2
- net GOUT: now also J1.2, J2.11 (GREEN)
- net ROUT: now also J1.1, J2.15 (RED/CHROMA)
- net GIN: now reaches C15.2, RV2.2
- net RO: now reaches C14.1
- net RO: now also R17.2
- net RIN: now reaches C14.2, RV1.2
- net BIN: now reaches C16.2, RV3.2
- net BO: now reaches R19.2
- net BO: now also C16.1
- net GO: now reaches R18.2
- net GO: now also C15.1
- net SYNCOUT renamed CSYNCO
- net CSYNCO: now also J2.20 (VIDIN/Sync), R10.2, R9.1
- new net: R26.2, U6.7 (VSOUT)
- new net: C32.1, C33.1, C34.2, R10.1
- new net: R25.2, U6.6 (HSOUT)
- new net: R24.2, U6.1 (REXT)
- new net +12V: R29.2
- new net +12V-1K: J2.8 (SW), R29.1
- new net 2.5V: J2.16 (BLNK), R27.2, R28.1
- new net GND1: C13.2, J1.10 (P10), J1.5
- new net GNDA: J1.6, J1.7, J1.8, J2.13 (RGND), J2.17 (VGND), J2.4 (AUGND), J2.5 (BGND), J2.9 (GGND)
- new net HSYNC: J1.13 (P13), R25.1
- new net SYNCIN: C34.1, U6.4 (VIN)
- new net VSYNC: J1.14 (P14), R26.1
- no-connect marks 7 -> 16
Other:
- note added: "Implementing Superimpose: ----------------------- 1. Feed external HSYNC / VSYNC into V9990 HRESET / VRESET pins for synchronisation 2. Combine external and internal R, G, B with an analog multiplexer, controlled by /Ys signal The principle is that the original external signal is passed through while /Ys is not superimposing."
- note added: "Loading Blank with 2.5V signals to the Monitor that the Scart is in RGB-mode."
- note added: "Sync Separator"
- note added: "Video Output Connectors"
- note removed: "Connectors"
- moved on the sheet: C14, C15, C16, C17, C19, C20, C21, Q1, R12, R13, R15, R17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
