File: Hardware/Kicad/TRH9000/TRH9000_VIDEO.kicad_sch (KiCad schematic)
At the start: 40 parts, among them J1 RGB, J2 Console5_SCART, Q1 BC817, U6 LMH1980

Commit message: More routing of the analog portion. Added 3D-models for the VGA and Scart connectors.
Parts:
- removed J1: RGB, LRJ:DSUB-Amphenol_L77HDE15SD1CH4RHNVGA, symbol LRJ-parts:Amphenol_L77HDE15SD1CH4RHNVGA
- added J1: Norcomp_200-015-263R001, LRJ:Norcomp_DSUB-15-HD_Female_Horizontal_SMD_P0.77x1.98mm, symbol LRJ-parts:Norcomp_200-015-263R001
- added R14: 75, Resistor_SMD:R_0603_1608Metric, symbol Device:R
- C2, C24: Price €0,14 -> (none)
- C34: Mounting Type SMD -> (none); Voltage Rating (none) -> 50V; Voltage Rating  50V -> (none)
Connections:
- net BOUT: now also J1.3 (BLUE)
- net GNDD: now also J1.10 (Sync_Ret/GND), J1.5 (GNDD)
- net GOUT: now also J1.2 (GREEN)
- net HSYNC: now also J1.13 (HSync)
- net ROUT: now also J1.1 (RED)
- net VGA_GND: now also J1.6 (GNDr), J1.7 (GNDg), J1.8 (GNDb)
- net VSYNC: now also J1.14 (VSync)
- net at R7.2: now also J1.SH
- net AUGND: now reaches C25.2, J2.14 (DATGND), J2.18 (BLNKGND), J2.4 (AUGND)
- net CSOUT: now reaches U6.8 (CSOUT)
- net CSOUT: now also R14.2
- net CSYNCO renamed ~{CSYNCA}
- net ~{CSYNCA}: no longer J2.20 (VIDIN/Sync)
- net Csync_ renamed ~{CSYNCA_}
- new net ~{CSYNCO}: J2.20 (VIDIN/Sync), R14.1
- no-connect marks 16 -> 15
Other:
- note added: "Loading SW with 12V sets the aspect ratio to 4:3"
- note removed: "IF = External Hreset + Vreset Then = superimpose"
- note removed: "Implementing Superimpose: ----------------------- 1. Feed external HSYNC / VSYNC into V9990 HRESET / VRESET pins for synchronisation 2. Combine external and internal R, G, B with an analog multiplexer, controlled by /Ys signal The principle is that the original external signal is passed through while /Ys is not superimposing."
- moved on the sheet: C17, C19, C20, C21, C32, C33, C34, Q1, R10, R11, R12, R13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

Commit message: Did a reroute of the analog / digital separation.
Did a reroute of the analog / digital separation.
Parts:
- removed C9: 47pF, Capacitor_SMD:C_0805_2012Metric, symbol Device:C
- removed R8: 2K2, Resistor_SMD:R_0805_2012Metric, symbol Device:R
- added U7: T.I_SN74CBT3257, trh9000:Texas_R-PDSO-G16_3.9x9.9mm, symbol TRH9000:T.I_SN74CBT3257
Connections:
- net SOUNDOUT: now reaches J2.6 (AIL/MONO)
- net B renamed Bm
- net Bm: now also U7.9 (3A)
- net G renamed Gm
- net Gm: now also U7.7 (2A)
- net R renamed Rm
- net Rm: now also U7.4 (1A)
- net REXT renamed REXTi
- net ~{CSYNC} renamed ~{CSYNCi}
- new net Be: U7.10 (3B2)
- new net Bi: U7.11 (3B1)
- new net Ge: U7.6 (2B2)
- new net Gi: U7.5 (2B1)
- new net Re: U7.3 (1B2)
- new net Ri: U7.2 (1B1)
- new net ~{YSe}: U7.1 (S)
- new net ~{YSi}: U7.15 (~{OE})
- no-connect marks 15 -> 17
Other:
- note added: "3. Sync Separator (internal)"
- note added: "6 lines of RGB. 1 line of YS (CS enable)"
- note added: "B1"
- note added: "B2"
- note added: "External signals"
- note added: "Function"
- note added: "Internal Signals"
- note added: "LEGEND: -------- CSYNCA = Amplified composite sync"
- note added: "MUX selection table:"
- note added: "Output = B1 port Output = B2 port Disconnect"
- note added: "S 0 1 x"
- note added: "V9958 (ext. VDP)"
- note added: "V9990 (int. VDP)"
- note added: "~{OE} 0 0 1"
- note removed: "3. Sync Separator"
- moved on the sheet: C13, C14, C15, C16, C17, C19, C2, C20, C21, C24, C25, C32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

Commit message: More routing - almost finished - only 29 more lines to go...
Parts:
- C2: footprint Capacitor_SMD:C_0805_2012Metric -> LRJ:C_0805_2012Metric_round_court
Changed lines of the file:
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@@
       (effects (font (size 1.143 1.143)) (justify left bottom) hide)
     )
-    (property "Footprint" "Capacitor_SMD:C_0805_2012Metric" (id 2) (at 281.94 226.06 0)
+    (property "Footprint" "LRJ:C_0805_2012Metric_round_court" (id 2) (at 281.94 226.06 0)
       (effects (font (size 0.508 0.508)) hide)
     )
