File: Hardware/Kicad/TRH9000/TRH9000.kicad_pcb (KiCad board)
At the start: 2 copper layers, 99.1 x 63.5 mm, 62 parts, among them J1 RGB, J100 MSX_SLOT_CONNECTOR, J2 S-Video, Q1 BC817, U1 V9990, U2 KM428C256, U3 KM428C256, U4 74HC138, U5 74HC32, U6 CXA2075M, X1 14.318Mhz, Y1 21.47727Mhz

Commit message: Merging in most recent upstream changes.
Parts:
- removed C18: 47pF, Capacitor_SMD:C_0805_2012Metric
- removed C22, C23, C24: 220uF, Capacitor_THT:CP_Radial_D5.0mm_P2.50mm
- removed C9: 100nF, Capacitor_SMD:C_0805_2012Metric
- removed J100: MSX_SLOT_CONNECTOR, msx:msx_cartridge
- removed R11: 4K7, Resistor_SMD:R_0805_2012Metric
- removed R14, R8: 2K2, Resistor_SMD:R_0805_2012Metric
- removed R16: 2K61, Resistor_SMD:R_0805_2012Metric
- removed R20: 43R, Resistor_SMD:R_0805_2012Metric
- removed R21, R22: 75R, Resistor_SMD:R_0805_2012Metric
- removed R23: 240R, Resistor_SMD:R_0805_2012Metric
- removed REF**: OSHW-Logo_11.4x12mm_SilkScreen, Symbol:OSHW-Logo_11.4x12mm_SilkScreen
- added BUS1: MSX_SLOT_EDGE-CON, trh9000:msx_cartridge, F.Cu at (152.9, 120.8)
- added C25: 1 µF, Capacitor_SMD:C_0805_2012Metric, F.Cu at (126.5, 110.0)
- added C26: 1 µF, Capacitor_SMD:C_0805_2012Metric, F.Cu at (122.5, 109.9)
- added C27: 1 µF, Capacitor_SMD:C_0805_2012Metric, B.Cu at (130.2, 110.6)
- added C28: 1 µF, Capacitor_SMD:C_0805_2012Metric, B.Cu at (166.9, 111.2)
- added C29: 0.1uF, Capacitor_SMD:C_0805_2012Metric, B.Cu at (163.4, 111.2)
- added C30: 1 µF, Capacitor_SMD:C_0805_2012Metric, B.Cu at (166.5, 101.2)
- added C31: 0.1uF, Capacitor_SMD:C_0805_2012Metric, B.Cu at (162.9, 101.3)
- added C32: 47pF, Capacitor_SMD:C_0805_2012Metric, B.Cu at (176.1, 94.7)
- added C33: 47pF, Capacitor_SMD:C_0805_2012Metric, B.Cu at (171.5, 94.7)
- added C34: 0.1µF, Capacitor_SMD:C_0805_2012Metric, B.Cu at (172.9, 88.9)
- added C35: 10uF, Capacitor_SMD:C_0805_2012Metric_Pad1.18x1.45mm_HandSolder, B.Cu at (166.1, 88.2)
- added C36: 0.1µF, Capacitor_SMD:C_0805_2012Metric, B.Cu at (166.1, 94.7)
- added Cart1: MSX-cartridge_dummy, trh9000:MSX-cart-dummy, F.Cu at (128.1, 151.4)
- added L3: 4.7µH, Inductor_SMD:L_0805_2012Metric, B.Cu at (160.5, 93.7)
- added R10: 100, Resistor_SMD:R_0805_2012Metric, B.Cu at (179.8, 87.9)
- added R24: 10k, Capacitor_SMD:C_0805_2012Metric, B.Cu at (150.2, 93.0)
- added R25: 100, Resistor_SMD:R_0805_2012Metric, B.Cu at (155.4, 93.0)
- added R26: 100, Resistor_SMD:R_0805_2012Metric, B.Cu at (152.7, 88.8)
- added R27: 100, Resistor_SMD:R_0603_1608Metric, F.Cu at (102.8, 19.7)
- added R28: 100, Resistor_SMD:R_0603_1608Metric, F.Cu at (107.8, 20.1)
- added R29: 1k, Resistor_SMD:R_0603_1608Metric, F.Cu at (111.9, 20.0)
- added R9: 75, Resistor_SMD:R_0805_2012Metric, B.Cu at (180.5, 94.8)
- C10, C11, C7: value 100nF -> 0.1uF
- C12, C5: value 100nF -> 0.1uF; moved to F.Cu
- C13: value 47pF -> 10µF; footprint Capacitor_THT:CP_Radial_D5.0mm_P2.50mm -> Capacitor_SMD:C_0805_2012Metric
- C2, L1, L2, R5: moved to F.Cu
- C3: footprint Capacitor_THT:CP_Radial_D5.0mm_P2.50mm -> Capacitor_SMD:C_0805_2012Metric
- C6: value 100nF -> 10nF
- C8: value 100nF -> 10nF; moved to F.Cu
- J2: value S-Video -> Console5_SCART; footprint Connector_PinHeader_2.54mm:PinHeader_1x04_P2.54mm_Vertical -> LRJ:SCART-21_Female_Horizontal_P1.905x2.54mm_EdgePinOffset10.7mm
- Q1, R12, R13, R15: moved to B.Cu
- U1: footprint trh9000:QFP-128_28x28_Pitch0.8mm -> trh9000:LQFP-128_28x28mm_P0.8mm
- U6: value CXA2075M -> LMH1980; footprint Package_SO:SOP-24_7.5x15.4mm_P1.27mm -> Package_SO:VSSOP-10_3x3mm_P0.5mm; moved to B.Cu
- X1: value 14.318Mhz -> 14.31818MHz; footprint Oscillator:Oscillator_DIP-8 -> Oscillator:Oscillator_DIP-14
- Y1: footprint Crystal:Crystal_HC50_Vertical -> Crystal:Crystal_HC49-U_Vertical
- moved C11 115.5 mm to (130.5, 109.9), turned to -90 degrees
- moved J2 97.6 mm to (124.1, 31.1)
- moved U7 93.4 mm to (156.2, 99.3)
- moved L1 91.4 mm to (171.9, 100.2)
- moved L2 91.2 mm to (171.8, 105.4), turned to 0 degrees
- moved C2 90.7 mm to (165.5, 101.0), turned to 180 degrees
- moved C17 89.0 mm to (173.7, 82.8), turned to 180 degrees
- moved R15 83.4 mm to (178.6, 82.2), turned to 180 degrees
- moved C3 79.8 mm to (165.6, 106.3), turned to 180 degrees
- moved R12 76.7 mm to (165.7, 81.7)
- moved U4 75.9 mm to (156.3, 109.2)
- moved R13 75.4 mm to (192.2, 81.2), turned to 180 degrees
- moved Q1 71.1 mm to (184.9, 83.2), turned to -90 degrees
- moved R3 56.9 mm to (186.9, 89.0)
- moved C1 51.6 mm to (179.6, 96.0)
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- renumbered U5 to U7
Connections:
- net /CLK renamed /SYS_CLK
- net /~{/INT} renamed /~{INT}
- net /~{/WAIT} renamed /~{WAIT}
- net Net-(C1-Pad1) renamed /VDP/X1
- net Net-(C14-Pad2) renamed /VIDEO/RIN
- net Net-(C15-Pad2) renamed /VIDEO/GIN
- net Net-(C16-Pad2) renamed /VIDEO/BIN
- net Net-(C4-Pad1) renamed /VDP/X2
- net Net-(R4-Pad2) renamed /VDP/VMREQ
- net Net-(U1-Pad38) renamed /VDP/~{V0_RAS}
- net Net-(U1-Pad39) renamed /VDP/~{V0_CAS}
- net Net-(U1-Pad40) renamed /VDP/~{V0_WE}
- net Net-(U1-Pad41) renamed /VDP/~{V0_TR}
- net Net-(U1-Pad42) renamed /VDP/~{V0_SC}
- net Net-(U1-Pad43) renamed /VDP/~{VO_SOE}
- net Net-(U1-Pad62) renamed /VDP/~{V1_RAS}
- net Net-(U1-Pad63) renamed /VDP/~{V1_CAS}
- net Net-(U1-Pad65) renamed /VDP/~{V1_WE}
- net Net-(U1-Pad66) renamed /VDP/~{V1_TR}
- net Net-(U1-Pad67) renamed /VDP/~{V1_SC}
- net Net-(U1-Pad68) renamed /VDP/~{V1_SOE}
- C11 pad 1: +5V -> GND
- C11 pad 2: GND -> +12V
- C12 pad 1: +5V -> -12V
- C13 pad 1: Net-(C13-Pad1) -> GND
- C13 pad 2: GND -> GND1
- C14 pad 1: Net-(C14-Pad1) -> /VIDEO/RO
- C15 pad 1: Net-(C15-Pad1) -> /VIDEO/GO
- C16 pad 1: Net-(C16-Pad1) -> /VIDEO/BO
- C8 pad 1: +5V -> GND
- C8 pad 2: GND -> +5V
- J1 pad 10: GND -> GND1
- J1 pad 13: /VIDEO/SYNCOUT -> /VIDEO/HSYNC
- J1 pad 14: unconnected-(J1-Pad14) -> /VIDEO/VSYNC
- J1 pad 5: GND -> GND1
- J1 pad 6: GND -> GNDA
- J1 pad 7: GND -> GNDA
- J1 pad 8: GND -> GNDA
- J2 pad 1: GND -> unconnected-(J2-Pad1)
- J2 pad 2: GND -> unconnected-(J2-Pad2)
- J2 pad 3: /VIDEO/YOUT -> unconnected-(J2-Pad3)
- J2 pad 4: /VIDEO/COUT -> GNDA
- L1 pad 1: GND -> +5V
- L1 pad 2: GNDA -> +5VA
- L2 pad 1: +5V -> GND
- L2 pad 2: +5VA -> GNDA
- R15 pad 1: /VIDEO/SYNCOUT -> /VIDEO/CSYNCO
- R17 pad 2: Net-(R17-Pad2) -> /VIDEO/RO
- R18 pad 2: Net-(R18-Pad2) -> /VIDEO/GO
- R19 pad 2: Net-(R19-Pad2) -> /VIDEO/BO
- R5 pad 2: Net-(R5-Pad2) -> /VDP/HRESET
- R6 pad 1: +5V -> /VDP/VRESET
- R6 pad 2: Net-(R6-Pad2) -> +5V
- U1 pad 105: Net-(R6-Pad2) -> /VDP/HRESET
- U1 pad 106: Net-(R5-Pad2) -> /VDP/VRESET
- U1 pad 113: Net-(U1-Pad113) -> /VDP/MCKIN
- U1 pad 2: /VDP/~{VDPW} -> /VDP/~{VDPR}
- U1 pad 3: /VDP/~{VDPR} -> /VDP/~{VDPW}
- U4 pad 4: /~{/IORQ} -> /~{IORQ}
- U4 pad 6: /~{/M1} -> /~{M1}
- U6 pad 1: GND -> Net-(R24-Pad2)
- U6 pad 10: Net-(C18-Pad1) -> unconnected-(U6-Pad10)
- U6 pad 2: Net-(C14-Pad1) -> GND
- U6 pad 3: Net-(C15-Pad1) -> +5VA
- U6 pad 4: Net-(C16-Pad1) -> /VIDEO/SYNCIN
- U6 pad 6: Net-(C13-Pad1) -> Net-(R25-Pad2)
- U7 pad 1: /~{/RD} -> /~{RD}
- U7 pad 4: /~{/WR} -> /~{WR}
- U7 pad 8: /VIDEO/SCIN -> /SCIN
- X1 pad 8: +5V -> /VDP/MCKIN
Routing:
- net +5V: track 0.00 -> 84.2 mm, vias 0 -> 11
- net /D6: track 0.00 -> 76.4 mm, vias 0 -> 2
- net /D4: track 0.00 -> 73.6 mm, vias 0 -> 2
- net /VDP/V1D3: track 0.00 -> 72.4 mm, vias 0 -> 2
- net /D7: track 0.00 -> 72.1 mm, vias 0 -> 1
- net /D2: track 0.00 -> 71.4 mm, vias 0 -> 2
- net /D5: track 0.00 -> 70.6 mm, vias 0 -> 1
- net /VDP/V1D2: track 0.00 -> 68.6 mm, vias 0 -> 2
- net /A2: track 0.00 -> 68.5 mm, vias 0 -> 2
- net /D3: track 0.00 -> 68.3 mm, vias 0 -> 1
- net /D0: track 0.00 -> 67.7 mm, vias 0 -> 2
- net /D1: track 0.00 -> 67.6 mm, vias 0 -> 1
- net GND: track 0.00 -> 67.1 mm, vias 0 -> 18
- net /A3: track 0.00 -> 66.3 mm, vias 0 -> 1
- net /A1: track 0.00 -> 66.3 mm, vias 0 -> 1
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- added copper zone on In2.Cu, net +5V
- added copper zone on In1.Cu, net GND
Other:
- board size 99.1 x 63.5 mm -> 110.2 x 63.5 mm
- copper layers 2 -> 4
