File: Hardware/Kicad/TRH9000/TRH9000.kicad_sch (KiCad schematic)
At the start: 6 parts, among them J100 MSX_SLOT_CONNECTOR, U4 74HC138, U5 74HC32

Commit message: Merging in most recent upstream changes.
Parts:
- removed C10, C11, C12: 100nF, Capacitor_SMD:C_0805_2012Metric, symbol Device:C
- removed J100: MSX_SLOT_CONNECTOR, msx:msx_cartridge, symbol Connector_Generic:Conn_02x25_Odd_Even
- added BUS1: MSX_SLOT_EDGE-CON, trh9000:msx_cartridge, symbol TRH9000:MSX_SLOT_EDGE-CON
- added C10, C11, C12: 0.1uF, Capacitor_SMD:C_0805_2012Metric, symbol LRJ-parts:C_CC0805JPX7R9BB104
- added C25, C26, C27: 1 µF, Capacitor_SMD:C_0805_2012Metric, symbol LRJ-parts:C_CL21B105KBFNNNF
- added Cart1: MSX-cartridge_dummy, trh9000:MSX-cart-dummy, symbol TRH9000:MSX-cartridge_dummy
- U4: symbol 74xx_IEEE:74LS138 -> TRH9000:74VHC138; MPN (none) -> 74HC138; Manufacturer (none) -> Toshiba Semiconductor and Storage
- U7: renamed from U5; symbol dk_Logic-Gates-and-Inverters:SN74HC32N -> TRH9000:T.I_SN74AHCT32D; Category Integrated Circuits (ICs) -> (none); DK_Datasheet_Link http://www.ti.com/general/docs/suppproductinfo.tsp?distId=1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 -> (none); DK_Detail_Page /product-detail/en/texas-instruments/SN74HC32N/296-1589-5-N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 -> https://www.digikey.se/en/products/detail/texas-instruments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; Digi-Key_PN 296-1589-5-ND -> (none); Family Logic - Gates and Inverters -> (none); MPN SN74HC32N -> 74HC32
Connections:
- net +12V: now also BUS1.48 (+12V), C11.2, C25.2
- net +5V: now also BUS1.45 (+5V), BUS1.47 (+5V), C10.1, C27.1; no longer U4.16 (VCC), U7.14 (VCC)
- net -12V: now also BUS1.50 (-12V), C12.1, C26.1
- net A0: now also BUS1.28 (A0)
- net A1: now also BUS1.27 (A1)
- net A10: now also BUS1.20 (A10)
- net A11: now also BUS1.19 (A11)
- net A12: now also BUS1.23 (A12)
- net A13: now also BUS1.26 (A13)
- net A14: now also BUS1.25 (A14)
- net A15: now also BUS1.18 (A15)
- net A2: now also BUS1.30 (A2)
- net A3: now also BUS1.29 (A3)
- net A4: now also BUS1.32 (A4)
- net A5: now also BUS1.31 (A5)
- net A6: now also BUS1.22 (A6)
- net A7: now also BUS1.21 (A7)
- net A8: now also BUS1.24 (A8)
- net A9: now also BUS1.17 (A9)
- net D0: now also BUS1.34 (D0)
- net D1: now also BUS1.33 (D1)
- net D2: now also BUS1.36 (D2~{})
- net D3: now also BUS1.35 (D3)
- net D4: now also BUS1.38 (D4)
- net D5: now also BUS1.37 (D5)
- net D6: now also BUS1.40 (D6)
- net D7: now also BUS1.39 (D7)
- net GND: now also BUS1.41 (GND), BUS1.43 (GND), C10.2, C11.1, C12.2, C25.1, C26.2, C27.2; no longer U4.8 (GND), U7.7 (GND)
- net SW1: now also BUS1.44 (SW1)
- net SW2: now also BUS1.46 (SW2)
- net ~{RESET}: now also BUS1.15 (~{RESET})
- net CLK renamed SYS_CLK
- net SYS_CLK: now also BUS1.42 (CLOCK)
- net VIDEO/SCIN renamed SCIN
- net ~{/IORQ} renamed ~{IORQ}
- net ~{IORQ}: now also BUS1.11 (~{IORQ})
- net ~{/M1} renamed ~{M1}
- net ~{M1}: now also BUS1.9 (~{M1})
- net ~{/RD} renamed ~{RD}
- net ~{RD}: now also BUS1.14 (~{RD})
- net ~{/WR} renamed ~{WR}
- net ~{WR}: now also BUS1.13 (~{WR})
- new net ~{BUSDIR}: BUS1.10 (~{BUSDIR})
- new net ~{CS12}: BUS1.3 (~{CS12})
- new net ~{CS1}: BUS1.1 (~{CS1})
- new net ~{CS2}: BUS1.2 (~{CS2})
- new net ~{INT}: BUS1.8 (~{INT})
- new net ~{MERQ}: BUS1.12 (~{MERQ})
- new net ~{RFSH}: BUS1.6 (~{RFSH})
- new net ~{SLTSL}: BUS1.4 (~{SLTSL})
- new net ~{WAIT}: BUS1.7 (~{WAIT})
- no-connect marks 10 -> 11
Other:
- added sheet Power (Power_v9990.kicad_sch)
- note added: "Cartridge-dummy - to allow testing of the mechanical form-factor."
- note added: "LEGEND: ------ VDP = Video Display Processor CLK = Clock SLTSL = Slot Select signal CS = Chip Select SYS_CLK = MSX System Clock"
- note added: "The MSX system-clock is often set to 3.58MHz - aka, the same as the sub-carrier clock of NTSC."
