File: Hardware/Kicad/TRH9000/TRH9000_VDP.kicad_sch (KiCad schematic)
At the start: 22 parts, among them U1 V9990, U2 KM428C256, U3 KM428C256, X1 14.318Mhz, Y1 21.47727Mhz

Commit message: Merging in most recent upstream changes.
Parts:
- removed C2, C5, C6, C7, C8, C9: 100nF, Capacitor_SMD:C_0805_2012Metric, symbol Device:C
- removed C3: 47uF, Capacitor_THT:CP_Radial_D5.0mm_P2.50mm, symbol Device:C_Polarized
- removed L1, L2: 4.7uH, Inductor_SMD:L_1206_3216Metric, symbol pspice:INDUCTOR
- added unit 3 of U1
- added unit 2 of U1
- U1: footprint trh9000:QFP-128_28x28_Pitch0.8mm -> trh9000:LQFP-128_28x28mm_P0.8mm; MPN (none) -> V9990; Manufacturer (none) -> Yamaha
- U2, U3: Manufacturer (none) -> Samsung Electronics Inc.; Status (none) -> OBSOLETE
- X1: value 14.318Mhz -> 14.31818MHz; footprint Oscillator:Oscillator_DIP-8 -> Oscillator:Oscillator_DIP-14; symbol Oscillator:CXO_DIP8 -> Oscillator:OCXO-14; Frequency (none) -> 14.31818MHz; MPN (none) -> CE3291-14.318180; Manufacturer (none) -> Crystek Corporation
Connections:
- net +5V: now also R6.2, X1.14 (Vcc); no longer R6.1, U1.123 (VCC), U1.27 (VCC), U1.53 (VCC), U1.81 (VCC), U1.97 (VCC), U2.1 (VCC), U2.20 (VCC), U3.1 (VCC), U3.20 (VCC), X1.8 (Vcc)
- net B: now also U1.95 (B/D1/CB1); no longer U1.95 (B/D31/CB1)
- net G: now also U1.94 (G/D2/CB2); no longer U1.94 (G/D2/CB2)
- net GND: now also X1.7 (GND); no longer U1.1 (GND), U1.100 (GND), U1.107 (GND), U1.118 (GND), U1.17 (GND), U1.32 (GND), U1.44 (GND), U1.64 (GND), U1.75 (GND), U1.86 (GND), U2.12 (VSS), U2.21 (VSS), U2.30 (VSS), U2.40 (VSS), U3.12 (VSS), U3.21 (VSS), U3.30 (VSS), U3.40 (VSS), X1.4 (GND)
- net R: now also U1.93 (R/D3/CB3); no longer U1.93 (R/D3/CB3)
- net V0A0: now also U1.26 (V0_A0/KA0); no longer U1.26 (V0A0/KA0)
- net V0A1: now also U1.25 (V0_A1/KA1); no longer U1.25 (V0A1/KA1)
- net V0A2: now also U1.24 (V0_A2/KA2); no longer U1.24 (V0A2/KA2)
- net V0A3: now also U1.23 (V0_A3/KA3); no longer U1.23 (V0A3/KA3)
- net V0A4: now also U1.22 (V0_A4/KA4); no longer U1.22 (V0A4/KA4)
- net V0A5: now also U1.21 (V0_A5/KA5); no longer U1.21 (V0A5/KA5)
- net V0A6: now also U1.20 (V0_A6/KA6); no longer U1.20 (V0A6/KA6)
- net V0A7: now also U1.19 (V0_A7/KA7); no longer U1.19 (V0A7/KA7)
- net V0A8: now also U1.18 (V0_A8/KA8); no longer U1.18 (V0A8/KA8)
- net V0D0: now also U1.36 (V0_D0/KD0); no longer U1.36 (V0D0/DK0)
- net V0D1: now also U1.35 (V0_D1/KD1); no longer U1.35 (V0D1/DK1)
- net V0D2: now also U1.34 (V0_D2/KD2); no longer U1.34 (V0D2/DK2)
- net V0D3: now also U1.33 (V0_D3/KD3); no longer U1.33 (V0D3/DK3)
- net V0D4: now also U1.31 (V0_D4/KD4); no longer U1.31 (V0D4/DK4)
- net V0D5: now also U1.30 (V0_D5/KD5); no longer U1.30 (V0D5/DK5)
- net V0D6: now also U1.29 (V0_D6/KD6); no longer U1.29 (V0D6/DK6)
- net V0D7: now also U1.28 (V0_D7/KD7); no longer U1.28 (V0D7/DK7)
- net V0S0: now also U1.52 (V0_S0); no longer U1.52 (V0S0)
- net V0S1: now also U1.51 (V0_S1); no longer U1.51 (V0S1)
- net V0S2: now also U1.50 (V0_S2); no longer U1.50 (V0S2)
- net V0S3: now also U1.49 (V0_S3); no longer U1.49 (V0S3)
- net V0S4: now also U1.48 (V0_S4); no longer U1.48 (V0S4)
- net V0S5: now also U1.47 (V0_S5); no longer U1.47 (V0S5)
- net V0S6: now also U1.46 (V0_S6); no longer U1.46 (V0S6)
- net V0S7: now also U1.45 (V0_S7); no longer U1.45 (V0S7)
- net V1A0: now also U1.80 (V1_A0); no longer U1.80 (V1A0)
- net V1A1: now also U1.79 (V1_A1); no longer U1.79 (V1A1)
- net V1A2: now also U1.78 (V1_A2); no longer U1.78 (V1A2)
- net V1A3: now also U1.77 (V1_A3); no longer U1.77 (V1A3)
- net V1A4: now also U1.76 (V1_A4); no longer U1.76 (V1A4)
- net V1A5: now also U1.74 (V1_A5); no longer U1.74 (V1A5)
- net V1A6: now also U1.73 (V1_A6); no longer U1.73 (V1A6)
- net V1A7: now also U1.72 (V1_A7); no longer U1.72 (V1A7)
- net V1A8: now also U1.71 (V1_A8); no longer U1.71 (V1A8)
- net V1D0: now also U1.82 (V1_D0); no longer U1.82 (V1D0)
- net V1D1: now also U1.83 (V1_D1); no longer U1.83 (V1D1)
- net V1D2: now also U1.84 (V1_D2); no longer U1.84 (V1D2)
- net V1D3: now also U1.85 (V1_D3); no longer U1.85 (V1D3)
- net V1D4: now also U1.87 (V1_D4); no longer U1.87 (V1D4)
- net V1D5: now also U1.88 (V1_D5); no longer U1.88 (V1D5)
- net V1D6: now also U1.89 (V1_D6); no longer U1.89 (V1D6)
- net V1D7: now also U1.90 (V1_D7); no longer U1.90 (V1D7)
- net V1S0: now also U1.61 (V1_S0); no longer U1.61 (V1S0)
- net V1S1: now also U1.60 (V1_S1); no longer U1.60 (V1S1)
- net V1S2: now also U1.59 (V1_S2); no longer U1.59 (V1S2)
- net V1S3: now also U1.58 (V1_S3); no longer U1.58 (V1S3)
- net V1S4: now also U1.57 (V1_S4); no longer U1.57 (V1S4)
- net V1S5: now also U1.56 (V1_S5); no longer U1.56 (V1S5)
- net V1S6: now also U1.55 (V1_S6); no longer U1.55 (V1S6)
- net V1S7: now also U1.54 (V1_S7); no longer U1.54 (V1S7)
- net ~{CSYNC}: now also U1.102 (~{CSYNC/FLM}); no longer U1.102 (~{CSYNC}/FLM)
- net ~{VDPR}: now also U1.2 (~{CSW}); no longer U1.3 (~{CSR})
- net ~{VDPW}: now also U1.3 (~{CSR}); no longer U1.2 (~{CSW})
- net X2: now reaches C4.1, R3.1, Y1.2
- net X2: now also U1.99 (XTAL2); no longer U1.99 (XTAL2)
- net ~{V0_WE}: now reaches U3.13 (R~{WB}/~{WE})
- net ~{V0_WE}: now also U1.40 (~{V0_WE}); no longer U1.40 (~{V0WE})
- net ~{V0_RAS}: now reaches U3.14 (~{RAS})
- net ~{V0_RAS}: now also U1.38 (~{V0_RAS}); no longer U1.38 (~{V0RAS})
- net ~{V0_SC}: now reaches U3.2 (SC)
- net ~{V0_SC}: now also U1.42 (~{V0_SC}); no longer U1.42 (V0SC)
- net ~{V0_CAS}: now reaches U3.27 (~{CAS})
- net ~{V0_CAS}: now also U1.39 (~{V0_CAS}); no longer U1.39 (~{V0CAS})
- net ~{VO_SOE}: now reaches U3.35 (~{SE})
- net ~{VO_SOE}: now also U1.43 (~{V0_SOE}); no longer U1.43 (~{V0SOE})
- net ~{V0_TR}: now reaches U3.7 (~{DT}/~{OE})
- net ~{V0_TR}: now also U1.41 (~{V0_TR/OE}); no longer U1.41 (~{V0TR}/~{OE})
- net X1: now reaches C1.1, R3.2, Y1.1
- net X1: now also U1.98 (XTAL1); no longer U1.98 (XTAL1)
- net ~{V1_WE}: now reaches U2.13 (R~{WB}/~{WE})
- net ~{V1_WE}: now also U1.65 (~{V1_WE}); no longer U1.65 (~{V1WE})
- net ~{V1_RAS}: now reaches U2.14 (~{RAS})
- net ~{V1_RAS}: now also U1.62 (~{V1_RAS}); no longer U1.62 (~{V1RAS})
- net ~{V1_SC}: now reaches U2.2 (SC)
- net ~{V1_SC}: now also U1.67 (V1_SC); no longer U1.67 (V1SC)
- net ~{V1_CAS}: now reaches U2.27 (~{CAS})
- net ~{V1_CAS}: now also U1.63 (~{V1_CAS}); no longer U1.63 (~{V1CAS})
- net ~{V1_SOE}: now reaches U2.35 (~{SE})
- net ~{V1_SOE}: now also U1.68 (~{V1_SOE}); no longer U1.68 (~{V1SOE})
- net ~{V1_TR}: now reaches U2.7 (~{DT}/~{OE})
- net ~{V1_TR}: now also U1.66 (~{V1_TR/OE}); no longer U1.66 (~{V1TR}/~{OE})
- net HRESET: now reaches R5.2
- net HRESET: now also U1.105 (~{HRESET}/CB4); no longer U1.106 (~{VRESET}/CB5)
- net VMREQ: now reaches R4.2, U1.124 (~{VMREQ})
- removed net +5VA: U1.96 (AVCC)
- removed net GNDA: U1.92 (AGND)
- new net MCKIN: U1.113 (MCKIN), X1.8 (OUT)
- new net VRESET: R6.1, U1.106 (~{VRESET}/CB5)
Other:
- note added: "VGA clocks: ------------- 640x400 (70Hz) - 25.175 MHz 640x480 (60Hz) - 25.175 MHz Pal clocks: ------------- 704x576 (50Hz) - 4.43361875 MHz NTSC clocks: -------------- 704x480 (60Hz) - 3.579545 MHz"
- note added: "VRAM"
- note added: "Video Display Processor"
- moved on the sheet: C1, C4, R1, R2, R3, R4, R5, R6, X1, Y1
