File: Hardware/TRH9000D-AA/TRH9000D-AA.kicad_sch (KiCad schematic)
At the start: 22 parts, among them J5 DIN-8_SD-80BV, U4 74VHC138, U5 T.I_SN74AHCT32D, U8 LMH1980

Commit message: Finished rerouting the AA-variant, and replaced the fuses with SMD-ones.
Parts:
- removed J5: DIN-8_SD-80BV, LRJ:Jack_DIN_CUI_SD-80BV_Vertical, symbol LRJ-parts:DIN-8_SD-80BV
- removed U5: T.I_SN74AHCT32D, trh9000:Texas_R-PDSO-G14_3.6x4.4mm, symbol TRH9000:T.I_SN74AHCT32D
- added J3: Norcomp_200-015-263R001, LRJ:Norcomp_DSUB-15-HD_Female_Horizontal_SMD_P0.77x1.98mm, symbol LRJ-parts:Norcomp_200-015-263R001
- added LOGO2: Logo_MSX, Ultra-MSX:Logo_MSX_10x3, symbol Ultra-MSX:Logo_MSX
- added U5: T.I_SN74LVC2G32DCTR, Package_SO:SSOP-8_2.95x2.8mm_P0.65mm, symbol TRH9000:T.I_SN74LVC2G32DCTR
- BUS1: value MSX-CONN_L-P -> MSX-CONN_L-P_v2; footprint trh9000:msx_edge-conn-LP -> trh9000:msx_edge-conn-LP_v2; symbol TRH9000:MSX-CONN_L-P -> TRH9000:MSX-CONN_L-P_v2
- C22, C42: value 47pF -> C_CC0603JRNPO9BN470; symbol Device:C -> LRJ-parts:C_CC0603JRNPO9BN470; Capacitance (none) -> 47pF; MPN (none) -> CC0603JRNPO9BN470; Manufacturer (none) -> Yageo; Mounting type (none) -> SMD; Operating Temperature (none) -> -55°C ~ 125°C; Status (none) -> Active; Temperature Coefficient  (none) -> C0G; Voltage rating (none) -> 50V
- C43: value 47pF -> C_CC0603JRNPO9BN470; footprint LRJ:C_0603_1608Metric_round_court -> Capacitor_SMD:C_0603_1608Metric; symbol Device:C -> LRJ-parts:C_CC0603JRNPO9BN470; Capacitance (none) -> 47pF; MPN (none) -> CC0603JRNPO9BN470; Manufacturer (none) -> Yageo; Mounting type (none) -> SMD; Operating Temperature (none) -> -55°C ~ 125°C; Status (none) -> Active; Temperature Coefficient  (none) -> C0G; Voltage rating (none) -> 50V
- C44: footprint LRJ:C_0603_1608Metric_round_court -> Capacitor_SMD:C_0603_1608Metric_Pad1.08x0.95mm_HandSolder; Mounting type (none) -> SMD
- LOGO1: now left out of the parts list
- R22: value 75 -> R_ERJ-PA3F75R0V; footprint Resistor_SMD:R_0603_1608Metric -> LRJ:R_0603_1608Metric_roundcourt; symbol Device:R -> LRJ-parts:R_ERJ-PA3F75R0V; MPN (none) -> ERJ-PA3F75R0V; Manufacturer (none) -> Panasonic Electronic Components; Mounting type (none) -> SMD; Operating Temperature  (none) -> -55°C to +155°C; Resistance (none) -> 75Ω; Status (none) -> Active; Temperature coeffecient (none) -> ±100ppm/°C; Voltage rating (none) -> 49V
- R23: value 100 -> R_CRGP0603F220R; footprint LRJ:R_0603_1608Metric_roundcourt -> Resistor_SMD:R_0603_1608Metric; symbol Device:R -> LRJ-parts:R_CRG0603F100R; MPN (none) -> CRGP0603F220R; Manufacturer (none) -> TE Connectivity; Operating Temperature  (none) -> -55°C to 125°C; Power (Watts)  (none) -> 0.1W, 1/10W; Resistance (none) -> 100Ω; Status (none) -> Active
- R31, R32: value 100 -> R_CRGP0603F220R; symbol Device:R -> LRJ-parts:R_CRG0603F100R; MPN (none) -> CRGP0603F220R; Manufacturer (none) -> TE Connectivity; Operating Temperature  (none) -> -55°C to 125°C; Power (Watts)  (none) -> 0.1W, 1/10W; Resistance (none) -> 100Ω; Status (none) -> Active
Connections:
- net Be: now also J3.3 (BLUE)
- net GND: now also R22.1; no longer R22.2
- net GNDe: now also J3.10 (Sync_Ret/GND), J3.5 (GNDD), J3.6 (GNDr), J3.7 (GNDg), J3.8 (GNDb)
- net Ge: now also J3.2 (GREEN)
- net Re: now also J3.1 (RED)
- net SOUNDOUT: now also J3.4 (ID_Bit2)
- net VDP/~{VDPR}: now also U5.7 (1Y)
- net VDP/~{VDPW}: now also U5.3 (2Y)
- net ~{CSYNCe}: now also R22.2, J3.14 (VSync); no longer R22.1
- net ~{RD}: now also U5.1 (1A)
- net ~{WR}: now also U5.5 (2A)
- net ~{Y6}: now also U5.2 (1B), U5.6 (2B)
- net at R8.2: now also J3.SH
- no-connect marks 34 -> 24
Other:
- sheet VIDEO ports: added none; removed ~{YSe}
- note added: "1.1. External RGB-input"
- note removed: "1.1. MSX standard RGB connector"
- moved on the sheet: C41, R22, R8
