File: Hardware/TRH9000D-AA/TRH9000_VIDEO.kicad_sch (KiCad schematic)
At the start: 40 parts, among them J1 Norcomp_200-015-263R001, J2 Console5_SCART, Q1 BC817, U6 LMH1980, U7 T.I_SN74CBT3257

Commit message: Finished rerouting the AA-variant, and replaced the fuses with SMD-ones.
Parts:
- removed Q1: BC817, Package_TO_SOT_SMD:SOT-23, symbol Transistor_BJT:BC817
- removed R12: 1K, Resistor_SMD:R_0805_2012Metric, symbol Device:R
- removed R13: 100R, Resistor_SMD:R_0805_2012Metric, symbol Device:R
- removed R15: 220R, Resistor_SMD:R_0805_2012Metric, symbol Device:R
- removed R27, R28: 100, Resistor_SMD:R_0603_1608Metric, symbol Device:R
- removed RV1, RV2, RV3: 500R, Potentiometer_SMD:Potentiometer_Bourns_3314G_Vertical, symbol Device:R_Potentiometer_Trim
- added C50, C51: C_TCJB227, Capacitor_Tantalum_SMD:CP_EIA-3528-15_AVX-H, symbol LRJ-parts:C_TCJB227
- added C59: C_GRM188D71A106KA73D, Capacitor_SMD:C_0603_1608Metric, symbol LRJ-parts:C_GRM188D71A106KA73D
- added L3: L_MLZ2012M4R7HT000, Inductor_SMD:L_0805_2012Metric, symbol LRJ-parts:L_MLZ2012M4R7HT000
- added R12, R40: R_RC0603FR-0710KL, LRJ:R_0603_1608Metric_roundcourt, symbol LRJ-parts:R_RC0603FR-0710KL
- added R13, R15, R41, R42, R43, R44: R_ERJ-PA3F75R0V, LRJ:R_0603_1608Metric_roundcourt, symbol LRJ-parts:R_ERJ-PA3F75R0V
- added R33, R35, R36, R37, R38, R39: R_CRCW08054K99FKEAHP, Resistor_SMD:R_0805_2012Metric_Pad1.20x1.40mm_HandSolder, symbol LRJ-parts:R_CRCW08054K99FKEAHP
- added R47 (x2): R_CRGP0603F220R, Resistor_SMD:R_0603_1608Metric, symbol LRJ-parts:R_CRG0603F100R
- added RV1, RV2, RV3: R_3314G-2-201E, LRJ:Potentiometer_Bourns_3314G_Vertical_lrj, symbol LRJ-parts:R_3314G-2-201E
- added U11: THS7374-lrj, Package_SO:TSSOP-14_4.4x5mm_P0.65mm, symbol LRJ-parts:THS7374-lrj
- C2: value C_CC0805JPX7R9BB104 -> C_CL10B104KB8NNNL; footprint LRJ:C_0805_2012Metric_round_court -> Capacitor_SMD:C_0603_1608Metric_Pad1.08x0.95mm_HandSolder; symbol LRJ-parts:C_CC0805JPX7R9BB104 -> LRJ-parts:C_CL10B104KB8NNNL; Capacitance 0.1uF -> (none); Capacitance  (none) -> 0,1µF; DK_Datasheet (none) -> https://media.digikey.com/pdf/Data%20Sheets/Samsung%20PDFs/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; MPN CC0805JPX7R9BB104 -> CL10B104KB8NNNL; Manufacturer Yageo -> Samsung Electro-Mechanics; Mouser datasheet https://www.mouser.se/datasheet/2/427/vjcommercialseries-17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 -> (none); Operating Temperature  (none) -> -55°C to +125°C; Package (none) -> 1608 Metric; Status Active -> (none); Tolerance (none) -> ±10%; Voltage Rating (none) -> 50V; Voltage rating 50V -> (none)
- C32, C33, C40: value 47pF -> C_CC0603JRNPO9BN470; symbol Device:C -> LRJ-parts:C_CC0603JRNPO9BN470; Capacitance (none) -> 47pF; MPN (none) -> CC0603JRNPO9BN470; Manufacturer (none) -> Yageo; Mounting type (none) -> SMD; Operating Temperature (none) -> -55°C ~ 125°C; Status (none) -> Active; Temperature Coefficient  (none) -> C0G; Voltage rating (none) -> 50V
- C34: Mounting type (none) -> SMD
- R10, R25, R26: value 100 -> R_CRGP0603F220R; symbol Device:R -> LRJ-parts:R_CRG0603F100R; MPN (none) -> CRGP0603F220R; Manufacturer (none) -> TE Connectivity; Operating Temperature  (none) -> -55°C to 125°C; Power (Watts)  (none) -> 0.1W, 1/10W; Resistance (none) -> 100Ω; Status (none) -> Active
- R14, R9: value 75 -> R_ERJ-PA3F75R0V; footprint Resistor_SMD:R_0603_1608Metric -> LRJ:R_0603_1608Metric_roundcourt; symbol Device:R -> LRJ-parts:R_ERJ-PA3F75R0V; MPN (none) -> ERJ-PA3F75R0V; Manufacturer (none) -> Panasonic Electronic Components; Mounting type (none) -> SMD; Operating Temperature  (none) -> -55°C to +155°C; Resistance (none) -> 75Ω; Status (none) -> Active; Temperature coeffecient (none) -> ±100ppm/°C; Voltage rating (none) -> 49V
- R17, R18, R19: value 75R -> R_ERJ-PA3F75R0V; footprint Resistor_SMD:R_0805_2012Metric -> LRJ:R_0603_1608Metric_roundcourt; symbol Device:R -> LRJ-parts:R_ERJ-PA3F75R0V; MPN (none) -> ERJ-PA3F75R0V; Manufacturer (none) -> Panasonic Electronic Components; Mounting type (none) -> SMD; Operating Temperature  (none) -> -55°C to +155°C; Resistance (none) -> 75Ω; Status (none) -> Active; Temperature coeffecient (none) -> ±100ppm/°C; Voltage rating (none) -> 49V
- R29: value 1k -> R_ERA-3VRW1001V; footprint Resistor_SMD:R_0603_1608Metric -> Resistor_SMD:R_0603_1608Metric_Pad0.98x0.95mm_HandSolder; symbol Device:R -> LRJ-parts:R_ERA-3VRW1001V; Details (none) -> https://na.industrial.panasonic.com/products/resistors/smd-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; MPN (none) -> ERA-3VRW1001V; Manufacturer (none) -> Panasonic; Operating temperature (none) -> -55C to +155C; Resistance (none) -> 1kΩ; Status (none) -> Active; Tolerance (none) -> ±0.05%; Voltage rating (none) -> 75V
- U7: value T.I_SN74CBT3257 -> AD8188; footprint trh9000:Texas_R-PDSO-G16_3.9x9.9mm -> Package_SO:TSSOP-24_4.4x7.8mm_P0.65mm; symbol TRH9000:T.I_SN74CBT3257 -> LRJ-parts:AD8188; MPN SN74CBT3257DR -> AD8188ARUZ; Manufacturer Texas Instruments -> Analog Devices Inc.
Connections:
- net ~{YSe} is gone; now on net Ri: U7.1 (IN0A)
- net +12V-1K: now also R29.2; no longer R29.1
- net +12VA: now also R29.1; no longer R29.2
- net +5VA: now also L3.1, R40.1, R47.1
- net 2.5VA: now also R47.1, R47.2
- net BIN: now also RV3.2 (Wiper)
- net BO: now also R19.1; no longer R19.2
- net BO_: now also R19.2; no longer R19.1
- net Be: now also U7.8 (IN2B), R36.2; no longer U7.10 (3B2)
- net Bi: now also U7.5 (IN2A), R39.2; no longer U7.11 (3B1)
- net Bm: now also U7.20 (OUT0), RV3.3 (CW); no longer U7.9 (3A)
- net GIN: now also RV2.2 (Wiper)
- net GND: now also R9.1, C59.1, R12.2, R13.2, R15.2, R41.2, R47.2, RV1.1 (CCW), RV2.1 (CCW), RV3.1 (CCW); no longer R9.2
- net GO: now also R18.1; no longer R18.2
- net GO_: now also R18.2; no longer R18.1
- net Ge: now also U7.10 (IN1B), R35.2; no longer U7.6 (2B2)
- net Gi: now also U7.3 (IN1A), R38.2; no longer U7.5 (2B1)
- net Gm: now also U7.16 (OUT2), RV2.3 (CW); no longer U7.7 (2A)
- net RIN: now also RV1.2 (Wiper)
- net RO: now also R17.1; no longer R17.2
- net RO_: now also R17.2; no longer R17.1
- net Re: now also U7.12 (IN0B), R33.2; no longer U7.3 (1B2)
- net Ri: now also R37.2; no longer U7.2 (1B1)
- net Rm: now also U7.18 (OUT1), RV1.3 (CW); no longer U7.4 (1A)
- net ~{CSYNCA}: now also C17.2, J2.20 (VIDIN/Sync); no longer R10.2, R9.1
- net ~{CSYNCO}: now also U11.1 (CH1_IN); no longer J2.20 (VIDIN/Sync)
- net ~{CSYNCi}: now also R10.2, R9.2
- net ~{YSi}: now also U7.22 (SEL_A/~{B}); no longer U7.15 (~{OE})
- net ~{CSYNCA}_: now reaches C17.1
- net ~{CSYNCA}_: now also R42.1
- net +5VL: now reaches J1.9 (DC_5V)
- net +5VL: now also C59.2, L3.2
- net HSYNC renamed HSYNCA
- net HSYNCA: now also C50.2; no longer R25.1
- net VSYNC renamed VSYNCA
- net VSYNCA: now also C51.2; no longer R26.1
- new net: R12.1, U11.11 (CH4_OUT), U11.4 (CH4_IN), U11.6 (DISABLE), U11.9 (BYPASS)
- new net HSYNCA_: C50.1, R43.1
- new net HSYNCO: R25.1, U11.2 (CH2_IN)
- new net HSYNC_: R15.1, R43.2, U11.13 (CH2_OUT)
- new net OE_MUX: R40.2, U7.23 (OE)
- new net VMID: R33.1, R35.1, R36.1, R37.1, R38.1, R39.1
- new net VSYNCA_: C51.1, R44.1
- new net VSYNCO: R26.1, U11.3 (CH3_IN)
- new net VSYNC_: R41.1, R44.2, U11.12 (CH3_OUT)
- new net ~{CSYNC}_: R13.1, R42.2, U11.14 (CH1_OUT)
- no-connect marks 17 -> 13
Other:
- note added: "1. Video MUX (w. amp)"
- note added: "2. RGB-coupling"
- note added: "4. Sync Amplifier"
- note added: "A"
- note added: "B"
- note added: "High-Z High-Z A port B port"
- note added: "Output"
- note added: "SEL A/~{B} 0 1 1 0"
- note added: "~{OE} 0 0 1 1"
- note removed: "1. RGB-input"
- note removed: "2. CSync Amplifier"
- note removed: "B1"
- note removed: "B2"
- note removed: "Function"
- note removed: "Output = B1 port Output = B2 port Disconnect"
- note removed: "S 0 1 x"
- note removed: "~{OE} 0 0 1"
- moved on the sheet: C13, C19, C20, C21, C24, C25, C34, J1, J2, R10, R11, R14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
