File: Hardware/TRH9000D-AB/TRH9000_VDP.kicad_sch (KiCad schematic)
At the start: 23 parts, among them J3 Conn_01x05_Female, J6 Conn_01x04_Female, U1 V9990, U2 KM428C256, U3 KM428C256, U9 SST39SF010A-lrj, X1 Crystek_CE3291, Y1 Y_HCM4921477270ABJT

Commit message: Finished rerouting the AA-variant, and replaced the fuses with SMD-ones.
Parts:
- added J4: Conn_01x05_Male, Connector_PinHeader_1.27mm:PinHeader_1x05_P1.27mm_Vertical, symbol Connector:Conn_01x05_Male
- added J7: Conn_01x05_Female, Connector_PinHeader_1.27mm:PinHeader_1x05_P1.27mm_Vertical, symbol Connector:Conn_01x05_Male
- added LOGO3: Logo_Open_Hardware_Small, Symbol:OSHW-Logo2_14.6x12mm_SilkScreen, symbol Graphic:Logo_Open_Hardware_Small
- J6: value Conn_01x04_Female -> Conn_01x05_Female; footprint Connector_PinSocket_1.27mm:PinSocket_1x04_P1.27mm_Vertical -> Connector_PinSocket_1.27mm:PinSocket_1x05_P1.27mm_Vertical; symbol Connector:Conn_01x04_Female -> Connector:Conn_01x05_Female
Connections:
- net +5VA: now also J6.5 (Pin_5), J4.5 (Pin_5), J7.5 (Pin_5)
- net B: now also J7.4 (Pin_4)
- net G: now also J7.3 (Pin_3)
- net GND: now also J4.2 (Pin_2), J7.1 (Pin_1)
- net R: now also J7.2 (Pin_2)
- net V9958_HSYNC: now also J4.3 (Pin_3)
- net V9958_VSYNC: now also J4.4 (Pin_4)
- net ~{CSYNCi}: now also J4.1 (Pin_1)
Other:
- moved on the sheet: C52, C53, C54, J3, R38, R39, R40
